Commit message: minor update

File: my_robot/robot_model/urdf/my_robot_model.urdf (robot description, URDF)
Before this commit: robot my_robot, 7 links, 6 joints
Joints:
- joint left_wheel_joint: origin xyz=0.2825 0.125 -0.15 rpy=1.5708 0 0 -> xyz=0.2825 0.125 -0.15 rpy=-1.5708 0 0
- joint right_wheel_joint: origin xyz=0.2825 -0.125 -0.15 rpy=1.5708 0 0 -> xyz=0.2825 -0.125 -0.15 rpy=-1.5708 0 0
